File: corne-light-bt-mx/corne-light-bt-mx_36.kicad_pcb (KiCad board)
At the start: 2 copper layers, 255.6 x 91.4 mm, 97 parts, among them SW10 SW_PUSH, SW11 SW_PUSH, SW12 SW_PUSH, SW14 SW_PUSH, SW15 SW_PUSH, SW16 SW_PUSH, SW17 SW_PUSH, SW18 SW_PUSH, SW19 SW_PUSH, SW2 SW_PUSH, SW20 SW_PUSH, SW21 SW_PUSH, SW22 SW_PUSH, SW23 SW_PUSH, SW24 SW_PUSH, SW25 SW_PUSH, SW26 SW_PUSH, SW27 SW_PUSH, SW28 SW_PUSH, SW29 SW_PUSH, SW3 SW_PUSH, SW30 SW_PUSH, SW31 SW_PUSH, SW32 SW_PUSH, SW33 SW_PUSH, SW34 SW_PUSH, SW35 SW_PUSH, SW36 SW_PUSH, SW37 SW_PUSH, SW38 SW_PUSH, SW39 SW_PUSH, SW4 SW_PUSH, SW40 SW_PUSH, SW41 SW_PUSH, SW42 SW_PUSH, SW5 SW_PUSH, SW6 SW_PUSH, SW8 SW_PUSH, SW9 SW_PUSH, U1 NiceNano!, U2 NiceNano!

Commit message: Corne36 work
Parts:
- added D1: D, Diode_SMD:D_SOD-123, B.Cu at (29.9, 45.9)
- added D13: D, Diode_SMD:D_SOD-123, B.Cu at (29.9, 83.9)
- added D7: D, Diode_SMD:D_SOD-123, B.Cu at (29.9, 64.9)
- added Ref**: Val**, PCM_kbd:spacer_m2, F.Cu at (31.7, 74.4)
- added Ref**: Val**, PCM_kbd:spacer_m2, F.Cu at (31.7, 55.4)
- added SW1: SW_PUSH, PCM_marbastlib-mx:SW_MX_1u, F.Cu at (22.2, 45.9)
- added SW13: SW_PUSH, PCM_marbastlib-mx:SW_MX_1u, F.Cu at (22.2, 83.9)
- added SW7: SW_PUSH, PCM_marbastlib-mx:SW_MX_1u, F.Cu at (22.2, 64.9)
Routing:
- net col0: track 34.0 -> 170.9 mm, vias 0 -> 1
- net row2: track 135.3 -> 150.9 mm
- net row1: track 147.4 -> 160.3 mm
- net row0: track 125.8 -> 137.4 mm
- net Net-(D1-Pad2): track 0.00 -> 7.34 mm
- net Net-(D7-Pad2): track 0.00 -> 6.84 mm
- net Net-(D13-Pad2): track 0.00 -> 6.67 mm
Other:
- board size 255.6 x 91.4 mm -> 274.7 x 91.4 mm
